File: eurorack/hardware/core_power/core_power.sch (KiCad schematic (older format))
At the start: 120 parts, among them J1 Power, J10 Jack, J11 Jack, J2 Serial, J3 SWD, J4 Jack, J5 Jack, J6 Jack, J7 Jack, J8 Jack, J9 Jack, SW2 Button, U1 STM32F405RGT6, U10 SC39-11SURKWA, U2 LM1117-3.3, U3 LM1117-3.3, U4 LM4040B10, U5 TLV320AIC23BPW, U6 TL072, U7 MCP6002, U8 MCP6002, U9 MCP6002, Y1 8MHz

Commit message: Add KiCad project with simple PCB
Signed-off-by: Petr Horacek <hrck@protonmail.com>
Parts:
- removed C33, C34: 100n, Capacitor_SMD:C_1206_3216Metric, symbol Device:C_Small
- removed C35, C37: 10u, Capacitor_SMD:CP_Elec_4x5.7, symbol Device:CP_Small
- removed C36, C38: 18p, Capacitor_SMD:C_0603_1608Metric, symbol Device:C_Small
- removed C39: 100n, Capacitor_SMD:C_0402_1005Metric, symbol Device:C_Small
- removed C40, C41, C42, C43, C44, C45, C46, C47, C48: 3n3, Capacitor_SMD:C_0603_1608Metric, symbol Device:C_Small
- removed J10, J11, J4, J5, J6, J7, J8, J9: Jack, Connector_Audio:Jack_3.5mm_QingPu_WQP-PJ398SM_Vertical_CircularHoles, symbol Connector:AudioJack2
- removed R10, R14: 1k, Resistor_SMD:R_0603_1608Metric, symbol Device:R_Small
- removed R11, R13, R19, R29, R7, R9: 47k, Resistor_SMD:R_0603_1608Metric, symbol Device:R_Small
- removed R12, R8: 6k8, Resistor_SMD:R_0603_1608Metric, symbol Device:R_Small
- removed R15: 10k, Resistor_SMD:R_0402_1005Metric, symbol Device:R_Small
- removed R16: 160, Resistor_SMD:R_0402_1005Metric, symbol Device:R_Small
- removed R17, R27: 180k, Resistor_SMD:R_0603_1608Metric, symbol Device:R_Small
- removed R18, R21, R25, R28, R30, R33: 100k, Resistor_SMD:R_0603_1608Metric, symbol Device:R_Small
- removed R20, R23, R24, R32: 120k, Resistor_SMD:R_0603_1608Metric, symbol Device:R_Small
- removed R22, R26, R31, R34: 20k, Resistor_SMD:R_0603_1608Metric, symbol Device:R_Small
- removed R35, R36, R37, R38, R39, R40, R41, R42: 365, Resistor_SMD:R_0603_1608Metric, symbol Device:R_Small
- removed RV1, RV2, RV3, RV4: 10k, Potentiometer_THT:Potentiometer_Alps_RK09L_Single_Vertical, symbol Device:R_POT
- removed SW2: Button, Button_Switch_THT:SW_PUSH_6mm, symbol Switch:SW_Push
- removed U10: SC39-11SURKWA, Display_7Segment:Sx39-1xxxxx, symbol Display_Character:SC39-11SRWA
- removed U6: TL072, Package_SO:SOIC-8_3.9x4.9mm_P1.27mm, symbol Amplifier_Operational:TL072
- removed U7, U8, U9: MCP6002, Package_SO:SOIC-8_3.9x4.9mm_P1.27mm, symbol Amplifier_Operational:MCP6002-xSN
- added J4: PowerConn, Connector_PinHeader_2.54mm:PinHeader_1x04_P2.54mm_Vertical, symbol Connector_Generic:Conn_01x04
- renumbered J3 to J2, J2 to J3
Connections:
- wire segments 444 -> 224
Other:
- note added: "Bus"
- note added: "TODO: One line of pins on each side"
- note removed: "-1.5 to 5.5"
- note removed: "-8.0 to 8.0"
- note removed: "Audio Output"
- note removed: "CV Input"
- note removed: "Connectivity"
- note removed: "Display"
- note removed: "Pin mapping:\n* PA1 - ADC1_IN1 - SCALE_POT\n* PA2 - ADC1_IN2 - VOCT_CV\n* PA5 - ADC1_IN5 - TABLE_CV\n* PA6 - ADC1_IN6 - RAMP_CV\n* PA7 - ADC1_IN7 - CAMP_CV\n* PA8 - GPIO_Output - DISPLAY_D\n* PA9 - GPIO_Output - DISPLAY_E\n* PA10 - GPIO_Output - DISPLAY_F\n* PA11 - GPIO_Output - DISPLAY_G\n* PA12 - GPIO_Output - DISPLAY_DP\n* PA13 - SYS_ITMS-SWDIO - SWDIO\n* PA14 - SYS_ITCK - SWCLK\n* PB3 - SYS_I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"
- note removed: "User Input"
- moved on the sheet: C1, C10, C11, C12, C13, C14, C15, C16, C17, C18, C19, C2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
