File: eurorack/hardware/core/core.sch (KiCad schematic (older format))
At the start: 50 parts, among them J1 ConnNW, J2 ConnSW, J3 ConnNE, J4 ConnSE, J5 Power, J6 SWD, SW1 Reset, SW2 Boot0, U1 STM32F427VGT6, U2 TLV320AIC23BPW, U3 LM1117F-3.3, U4 LM4040C10IDBZR, Y1 Crystal

Commit message: Add compatible heading to the BOM
Signed-off-by: Petr Horacek <hrck@protonmail.com>
Parts:
- C1, C2: LCSC (none) -> C1554
- C10, C20: LCSC (none) -> C52923
- C11, C12, C13, C14, C15, C16, C17, C18, C19, C21, C22, C23: LCSC (none) -> C1525
- C24: LCSC (none) -> C49678
- C3, C4, C7: LCSC (none) -> C23630
- C5, C6, C8, C9: LCSC (none) -> C129570
- D1, D2: LCSC (none) -> C8598
- FB1, FB2, FB3: LCSC (none) -> C1017
- R1: LCSC (none) -> C25118
- R2, R3: LCSC (none) -> C25744
- R4: LCSC (none) -> C22810
- R5, R6: LCSC (none) -> C25879
- R7, R8: LCSC (none) -> C17513
- SW1, SW2: LCSC (none) -> C115357
- U1: LCSC (none) -> C117815
- U2: LCSC (none) -> C9915
- U3: LCSC (none) -> C126019
- U4: LCSC (none) -> C201738
- Y1: LCSC (none) -> C115962
Changed lines of the file:
@@
 F 3 "http://www.st.com/st-web-ui/static/active/en/resource/technical/document/datasheet/DM00071990.pdf" H 3550 3650 50  0001 C CNN
 F 4 "C117815" H 3550 3650 50  0001 C CNN "LCSC Part #"
+F 5 "C117815" H 3550 3650 50  0001 C CNN "LCSC"
 	1    3550 3650
 	1    0    0    -1
@@
 F 3 "http://www.ti.com/lit/ds/symlink/tlv320aic23b.pdf" H 7075 3650 50  0001 C CNN
 F 4 "C9915" H 7075 3650 50  0001 C CNN "LCSC Part #"
+F 5 "C9915" H 7075 3650 50  0001 C CNN "LCSC"
 	1    7075 3650
 	1    0    0    -1
@@
 F 3 "http://www.ti.com/lit/ds/symlink/lm1117.pdf" H 9575 2575 50  0001 C CNN
 F 4 "C126019" H 9575 2575 50  0001 C CNN "LCSC Part #"
+F 5 "C126019" H 9575 2575 50  0001 C CNN "LCSC"
 	1    9575 2575
 	1    0    0    -1
@@
 F 3 "~" H 2200 1900 50  0001 C CNN
 F 4 "C23630" H 2200 1900 50  0001 C CNN "LCSC Part #"
+F 5 "C23630" H 2200 1900 50  0001 C CNN "LCSC"
 	1    2200 1900
 	1    0    0    -1
@@
 F 3 "~" H 9125 2750 50  0001 C CNN
 F 4 "C129570" H 9125 2750 50  0001 C CNN "LCSC Part #"
+F 5 "C129570" H 9125 2750 50  0001 C CNN "LCSC"
 	1    9125 2750
 	1    0    0    -1
@@
 F 3 "~" H 9925 2725 50  0001 C CNN
 F 4 "C129570" H 9925 2725 50  0001 C CNN "LCSC Part #"
+F 5 "C129570" H 9925 2725 50  0001 C CNN "LCSC"
 	1    9925 2725
 	1    0    0    -1
@@
 F 3 "~" H 10625 1425 50  0001 C CNN
 F 4 "C129570" H 10625 1425 50  0001 C CNN "LCSC Part #"
+F 5 "C129570" H 10625 1425 50  0001 C CNN "LCSC"
 	1    10625 1425
 	1    0    0    -1
@@
 F 3 "~" H 10625 1125 50  0001 C CNN
 F 4 "C129570" H 10625 1125 50  0001 C CNN "LCSC Part #"
+F 5 "C129570" H 10625 1125 50  0001 C CNN "LCSC"
 	1    10625 1125
 	1    0    0    -1
@@
 F 3 "~" H 8950 1075 50  0001 C CNN
 F 4 "C1017" H 8950 1075 50  0001 C CNN "LCSC Part #"
+F 5 "C1017" H 8950 1075 50  0001 C CNN "LCSC"
 	1    8950 1075
 	0    1    1    0
@@
 F 3 "~" H 8950 1475 50  0001 C CNN
 F 4 "C1017" H 8950 1475 50  0001 C CNN "LCSC Part #"
+F 5 "C1017" H 8950 1475 50  0001 C CNN "LCSC"
 	1    8950 1475
 	0    1    1    0
@@
 F 3 "~" H 10250 2725 50  0001 C CNN
 F 4 "C23630" H 10250 2725 50  0001 C CNN "LCSC Part #"
+F 5 "C23630" H 10250 2725 50  0001 C CNN "LCSC"
 	1    10250 2725
 	1    0    0    -1
@@
 F 3 "~" H 8950 2575 50  0001 C CNN
 F 4 "C22810" H 8950 2575 50  0001 C CNN "LCSC Part #"
+F 5 "C22810" H 8950 2575 50  0001 C CNN "LCSC"
 	1    8950 2575
 	0    1    1    0
@@
 F 3 "~" H 10575 2575 50  0001 C CNN
 F 4 "C1017" H 10575 2575 50  0001 C CNN "LCSC Part #"
+F 5 "C1017" H 10575 2575 50  0001 C CNN "LCSC"
 	1    10575 2575
 	0    1    1    0
@@
 F 3 "~" H 2875 7175 50  0001 C CNN
 F 4 "C52923" H 2875 7175 50  0001 C CNN "LCSC Part #"
+F 5 "C52923" H 2875 7175 50  0001 C CNN "LCSC"
 	1    2875 7175
 	1    0    0    -1
@@
 F 3 "~" H 3250 7175 50  0001 C CNN
 F 4 "C1525" H 3250 7175 50  0001 C CNN "LCSC Part #"
+F 5 "C1525" H 3250 7175 50  0001 C CNN "LCSC"
 	1    3250 7175
 	1    0    0    -1
@@
 F 3 "~" H 3650 7175 50  0001 C CNN
 F 4 "C1525" H 3650 7175 50  0001 C CNN "LCSC Part #"
+F 5 "C1525" H 3650 7175 50  0001 C CNN "LCSC"
 	1    3650 7175
 	1    0    0    -1
@@
 F 3 "~" H 4050 7175 50  0001 C CNN
 F 4 "C1525" H 4050 7175 50  0001 C CNN "LCSC Part #"
+F 5 "C1525" H 4050 7175 50  0001 C CNN "LCSC"
 	1    4050 7175
 	1    0    0    -1
@@
 F 3 "~" H 4450 7175 50  0001 C CNN
 F 4 "C1525" H 4450 7175 50  0001 C CNN "LCSC Part #"
+F 5 "C1525" H 4450 7175 50  0001 C CNN "LCSC"
 	1    4450 7175
 	1    0    0    -1
@@
 F 3 "~" H 4850 7175 50  0001 C CNN
 F 4 "C1525" H 4850 7175 50  0001 C CNN "LCSC Part #"
+F 5 "C1525" H 4850 7175 50  0001 C CNN "LCSC"
 	1    4850 7175
 	1    0    0    -1
@@
 F 3 "~" H 5250 7175 50  0001 C CNN
 F 4 "C1525" H 5250 7175 50  0001 C CNN "LCSC Part #"
+F 5 "C1525" H 5250 7175 50  0001 C CNN "LCSC"
 	1    5250 7175
 	1    0    0    -1
@@
 F 3 "~" H 5650 7175 50  0001 C CNN
 F 4 "C1525" H 5650 7175 50  0001 C CNN "LCSC Part #"
+F 5 "C1525" H 5650 7175 50  0001 C CNN "LCSC"
 	1    5650 7175
 	1    0    0    -1
@@
 F 3 "~" H 6050 7175 50  0001 C CNN
 F 4 "C1525" H 6050 7175 50  0001 C CNN "LCSC Part #"
+F 5 "C1525" H 6050 7175 50  0001 C CNN "LCSC"
 	1    6050 7175
 	1    0    0    -1
@@
 F 3 "~" H 6450 7175 50  0001 C CNN
 F 4 "C1525" H 6450 7175 50  0001 C CNN "LCSC Part #"
+F 5 "C1525" H 6450 7175 50  0001 C CNN "LCSC"
 	1    6450 7175
 	1    0    0    -1
@@
 F 3 "~" H 6175 2800 50  0001 C CNN
 F 4 "C25879" H 6175 2800 50  0001 C CNN "LCSC Part #"
+F 5 "C25879" H 6175 2800 50  0001 C CNN "LCSC"
 	1    6175 2800
 	1    0    0    -1
@@
 F 3 "~" H 5925 2800 50  0001 C CNN
 F 4 "C25879" H 5925 2800 50  0001 C CNN "LCSC Part #"
+F 5 "C25879" H 5925 2800 50  0001 C CNN "LCSC"
 	1    5925 2800
 	1    0    0    -1
@@
 F 3 "~" H 1875 1900 50  0001 C CNN
 F 4 "C23630" H 1875 1900 50  0001 C CNN "LCSC Part #"
+F 5 "C23630" H 1875 1900 50  0001 C CNN "LCSC"
 	1    1875 1900
 	1    0    0    -1
@@
 F 3 "~" H 1225 7150 50  0001 C CNN
 F 4 "C25744" H 1225 7150 50  0001 C CNN "LCSC Part #"
+F 5 "C25744" H 1225 7150 50  0001 C CNN "LCSC"
 	1    1225 7150
 	0    1    1    0
@@
 F 3 "~" H 1625 7350 50  0001 C CNN
 F 4 "C115357" H 1625 7150 50  0001 C CNN "LCSC Part #"
+F 5 "C115357" H 1625 7150 50  0001 C CNN "LCSC"
 	1    1625 7150
 	1    0    0    -1
@@
 F 3 "~" H 1725 6150 50  0001 C CNN
 F 4 "C25744" H 1725 6150 50  0001 C CNN "LCSC Part #"
+F 5 "C25744" H 1725 6150 50  0001 C CNN "LCSC"
 	1    1725 6150
 	0    1    1    0
@@
 F 3 "~" H 1325 6350 50  0001 C CNN
 F 4 "C115357" H 1325 6150 50  0001 C CNN "LCSC Part #"
+F 5 "C115357" H 1325 6150 50  0001 C CNN "LCSC"
 	1    1325 6150
 	1    0    0    -1
@@
 F 3 "~" H 1375 3250 50  0001 C CNN
 F 4 "C115962" H 1375 3250 50  0001 C CNN "LCSC Part #"
+F 5 "C115962" H 1375 3250 50  0001 C CNN "LCSC"
 	1    1375 3250
 	1    0    0    -1
@@
 F 3 "~" H 1175 3450 50  0001 C CNN
 F 4 "C1554" H 1175 3450 50  0001 C CNN "LCSC Part #"
+F 5 "C1554" H 1175 3450 50  0001 C CNN "LCSC"
 	1    1175 3450
 	1    0    0    -1
@@
 F 3 "~" H 1575 3450 50  0001 C CNN
 F 4 "C1554" H 1575 3450 50  0001 C CNN "LCSC Part #"
+F 5 "C1554" H 1575 3450 50  0001 C CNN "LCSC"
 	1    1575 3450
 	1    0    0    -1
@@
 F 3 "~" H 1175 3000 50  0001 C CNN
 F 4 "C25118" H 1175 3000 50  0001 C CNN "LCSC Part #"
+F 5 "C25118" H 1175 3000 50  0001 C CNN "LCSC"
 	1    1175 3000
 	1    0    0    -1
@@
 F 3 "~" H 6050 6425 50  0001 C CNN
 F 4 "C1525" H 6050 6425 50  0001 C CNN "LCSC Part #"
+F 5 "C1525" H 6050 6425 50  0001 C CNN "LCSC"
 	1    6050 6425
 	1    0    0    -1
@@
 F 3 "~" H 5650 6425 50  0001 C CNN
 F 4 "C1525" H 5650 6425 50  0001 C CNN "LCSC Part #"
+F 5 "C1525" H 5650 6425 50  0001 C CNN "LCSC"
 	1    5650 6425
 	1    0    0    -1
@@
 F 3 "~" H 5250 6425 50  0001 C CNN
 F 4 "C1525" H 5250 6425 50  0001 C CNN "LCSC Part #"
+F 5 "C1525" H 5250 6425 50  0001 C CNN "LCSC"
 	1    5250 6425
 	1    0    0    -1
@@
 F 3 "~" H 4875 6425 50  0001 C CNN
 F 4 "C52923" H 4875 6425 50  0001 C CNN "LCSC Part #"
+F 5 "C52923" H 4875 6425 50  0001 C CNN "LCSC"
 	1    4875 6425
 	1    0    0    -1
@@
 F 3 "http://www.ti.com/lit/ds/symlink/lm4040-n.pdf" H 7700 1050 50  0001 C CIN
 F 4 "C201738" H 7700 1050 50  0001 C CNN "LCSC Part #"
+F 5 "C201738" H 7700 1050 50  0001 C CNN "LCSC"
 	1    7700 1050
 	-1   0    0    1
@@
 F 3 "~" H 7700 1225 50  0001 C CNN
 F 4 "C49678" H 7700 1225 50  0001 C CNN "LCSC Part #"
+F 5 "C49678" H 7700 1225 50  0001 C CNN "LCSC"
 	1    7700 1225
 	0    1    1    0
@@
 F 3 "~" H 8250 1050 50  0001 C CNN
 F 4 "C17513" H 8250 1050 50  0001 C CNN "LCSC Part #"
+F 5 "C17513" H 8250 1050 50  0001 C CNN "LCSC"
 	1    8250 1050
 	0    1    1    0
@@
 F 3 "~" H 8250 1225 50  0001 C CNN
 F 4 "C17513" H 8250 1225 50  0001 C CNN "LCSC Part #"
+F 5 "C17513" H 8250 1225 50  0001 C CNN "LCSC"
 	1    8250 1225
 	0    1    1    0
@@
 F 3 "~" V 9150 1075 50  0001 C CNN
 F 4 "C8598" H 9150 1075 50  0001 C CNN "LCSC Part #"
+F 5 "C8598" H 9150 1075 50  0001 C CNN "LCSC"
 	1    9150 1075
 	1    0    0    -1
@@
 F 3 "~" V 9150 1475 50  0001 C CNN
 F 4 "C8598" H 9150 1475 50  0001 C CNN "LCSC Part #"
+F 5 "C8598" H 9150 1475 50  0001 C CNN "LCSC"
 	1    9150 1475
 	-1   0    0    1
